File: hardware/clockedIn.kicad_sch (KiCad schematic)
At the start: 1 part

Commit message: maybe i should commit the hardware files :sob:
Parts:
- added A1: RaspberryPi_Pico_W, Module:RaspberryPi_Pico_W_SMD_HandSolder, symbol MCU_Module:RaspberryPi_Pico_W
- added HV1: ~, symbol 170v:NCH8200HV
- added J1: Barrel_Jack_Switch, symbol Connector:Barrel_Jack_Switch
- added NX2, NX3, NX4, NX5, NX6: IN-12BORIGINAL, nixies-us_IN-12, symbol nixies-us:IN-12BORIGINAL
- added R1, R2, R3, R4, R5, R6: 22k, symbol Device:R
- added U1, U2, U3, U4, U5, U6, U7, U8, U9: TPIC6B595N, TPIC6B595N:DIP254P762X508-20, symbol TPIC6B595N:TPIC6B595N
Connections:
- net at NX1.A: now also R1.2
- new net: NX6.A, R6.2
- new net: U4.18 (SER_OUT), U5.3 (SER_IN)
- new net: U3.18 (SER_OUT), U4.3 (SER_IN)
- new net: NX5.A, R5.2
- new net: U8.18 (SER_OUT), U9.3 (SER_IN)
- new net: U7.18 (SER_OUT), U8.3 (SER_IN)
- new net: NX4.A, R4.2
- new net: U1.18 (SER_OUT), U2.3 (SER_IN)
- new net: U5.18 (SER_OUT), U6.3 (SER_IN)
- new net: NX3.A, R3.2
- new net: U6.18 (SER_OUT), U7.3 (SER_IN)
- new net: U2.18 (SER_OUT), U3.3 (SER_IN)
- new net: NX2.A, R2.2
- new net +5V: A1.39 (VSYS), J1.1, U1.2 (VCC), U1.8 (~SRCLR), U2.2 (VCC), U2.8 (~SRCLR), U3.2 (VCC), U3.8 (~SRCLR), U4.2 (VCC), U4.8 (~SRCLR), U5.2 (VCC), U5.8 (~SRCLR), U6.2 (VCC), U6.8 (~SRCLR), U7.2 (VCC), U7.8 (~SRCLR), U8.2 (VCC), U8.8 (~SRCLR), U9.2 (VCC), U9.8 (~SRCLR)
- new net 170v: HV1.3 (DC_OUT), R1.1, R2.1, R3.1, R4.1, R5.1, R6.1
- new net CLOCK: U1.13 (SRCK), U2.13 (SRCK), U3.13 (SRCK), U4.13 (SRCK), U5.13 (SRCK), U6.13 (SRCK), U7.13 (SRCK), U8.13 (SRCK), U9.13 (SRCK)
- new net DATA: U1.3 (SER_IN)
- new net GND: A1.13 (GND), A1.18 (GND), A1.23 (GND), A1.28 (GND), A1.3 (GND), A1.33 (AGND), A1.38 (GND), A1.8 (GND), HV1.2 (GND), J1.2, U1.10 (GND_2), U1.11 (GND), U1.19 (GND_3), U1.9 (~G), U2.10 (GND_2), U2.11 (GND), U2.19 (GND_3), U2.9 (~G), U3.10 (GND_2), U3.11 (GND), U3.19 (GND_3), U3.9 (~G), U4.10 (GND_2), U4.11 (GND), U4.19 (GND_3), U4.9 (~G), U5.10 (GND_2), U5.11 (GND), U5.19 (GND_3), U5.9 (~G), U6.10 (GND_2), U6.11 (GND), U6.19 (GND_3), U6.9 (~G), U7.10 (GND_2), U7.11 (GND), U7.19 (GND_3), U7.9 (~G), U8.10 (GND_2), U8.11 (GND), U8.19 (GND_3), U8.9 (~G), U9.10 (GND_2), U9.11 (GND), U9.19 (GND_3), U9.9 (~G)
- new net LATCH: U1.12 (RCK), U2.12 (RCK), U3.12 (RCK), U4.12 (RCK), U5.12 (RCK), U6.12 (RCK), U7.12 (RCK), U8.12 (RCK), U9.12 (RCK)
- no-connect marks 0 -> 19
Other:
- moved on the sheet: NX1

Commit message: hardware bump
Parts:
- added SW1: SW_SPDT, 500SSP3S1M6QEA:SW_500SSP3S1M6QEA, symbol Switch:SW_SPDT
- HV1: footprint (none) -> NCH8200HV:NCH8200HV
- NX1, NX2, NX3, NX4, NX5, NX6: footprint nixies-us_IN-12 -> nixies-us:nixies-us-IN-12-DSUB
- R1, R2, R3, R4, R5, R6: footprint (none) -> Resistor_THT:R_Axial_DIN0207_L6.3mm_D2.5mm_P10.16mm_Horizontal
Connections:
- net +5V: now also SW1.2 (B)
- net at HV1.1 (DC_IN): now also SW1.1 (A)
- no-connect marks 19 -> 20
Changed lines of the file:
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@@
 	)
 	(junction
+		(at 119.38 237.49)
+		(diameter 0)
+		(color 0 0 0 0)
+	)
+	(junction
 		(at 439.42 322.58)
 		(diameter 0)
@@
 	)
 	(no_connect
+		(at 135.89 240.03)
+	)
+	(no_connect
 		(at 191.77 312.42)
 	)
@@
 	(wire
 		(pts
+			(xy 135.89 234.95) (xy 139.7 234.95)
+		)
+		(stroke
+			(width 0)
+			(type default)
+		)
+	)
+	(wire
+		(pts
 			(xy 287.02 325.12) (xy 287.02 327.66)
 		)
@@
 	(wire
 		(pts
+			(xy 139.7 237.49) (xy 143.51 237.49)
+		)
+		(stroke
+			(width 0)
+			(type default)
+		)
+	)
+	(wire
+		(pts
 			(xy 344.17 294.64) (xy 337.82 294.64)
 		)
@@
 	(wire
 		(pts
+			(xy 119.38 237.49) (xy 125.73 237.49)
+		)
+		(stroke
+			(width 0)
+			(type default)
+		)
+	)
+	(wire
+		(pts
 			(xy 394.97 287.02) (xy 388.62 287.02)
 		)
@@
 	(wire
 		(pts
+			(xy 139.7 234.95) (xy 139.7 237.49)
+		)
+		(stroke
+			(width 0)
+			(type default)
+		)
+	)
+	(wire
+		(pts
 			(xy 336.55 297.18) (xy 344.17 297.18)
 		)
@@
 			)
 		)
-		(property "Footprint" ""
+		(property "Footprint" "Resistor_THT:R_Axial_DIN0207_L6.3mm_D2.5mm_P10.16mm_Horizontal"
 			(at 259.842 364.49 90)
 			(effects
@@
 	)
 	(symbol
+		(lib_id "Switch:SW_SPDT")
+		(at 130.81 237.49 0)
+		(unit 1)
+		(exclude_from_sim no)
+		(in_bom yes)
+		(on_board yes)
+		(dnp no)
+		(fields_autoplaced yes)
+		(property "Reference" "SW1"
+			(at 130.81 228.6 0)
+			(effects
+				(font
+					(size 1.27 1.27)
+				)
+			)
+		)
+		(property "Value" "SW_SPDT"
+			(at 130.81 231.14 0)
+			(effects
+				(font
+					(size 1.27 1.27)
+				)
+			)
+		)
+		(property "Footprint" "500SSP3S1M6QEA:SW_500SSP3S1M6QEA"
+			(at 130.81 237.49 0)
+			(effects
+				(font
+					(size 1.27 1.27)
+				)
+				(hide yes)
+			)
+		)
+		(property "Datasheet" "~"
+			(at 130.81 245.11 0)
+			(effects
+				(font
+					(size 1.27 1.27)
+				)
+				(hide yes)
+			)
+		)
+		(property "Description" "Switch, single pole double throw"
+			(at 130.81 237.49 0)
+			(effects
+				(font
+					(size 1.27 1.27)
+				)
+				(hide yes)
+			)
+		)
+		(pin "2"
+		)
+		(pin "1"
+		)
+		(pin "3"
+		)
+		(instances
+			(project ""
+				(path "/9262f813-14b2-4086-b979-00b2efb6aed1"
+					(reference "SW1")
+					(unit 1)
+				)
+			)
+		)
+	)
+	(symbol
 		(lib_id "power:+5V")
 		(at 388.62 285.75 0)
@@
 			)
 		)
-		(property "Footprint" "nixies-us_IN-12"
+		(property "Footprint" "nixies-us:nixies-us-IN-12-DSUB"
 			(at 249.682 364.49 0)
 			(effects
@@
 			)
 		)
-		(property "Footprint" ""
+		(property "Footprint" "Resistor_THT:R_Axial_DIN0207_L6.3mm_D2.5mm_P10.16mm_Horizontal"
 			(at 226.822 364.49 90)
 			(effects
@@
 			)
 		)
-		(property "Footprint" ""
+		(property "Footprint" "Resistor_THT:R_Axial_DIN0207_L6.3mm_D2.5mm_P10.16mm_Horizontal"
 			(at 74.422 364.49 90)
 			(effects
@@
 			)
 		)
-		(property "Footprint" ""
+		(property "Footprint" "Resistor_THT:R_Axial_DIN0207_L6.3mm_D2.5mm_P10.16mm_Horizontal"
 			(at 183.642 364.49 90)
 			(effects
@@
 			)
 		)
-		(property "Footprint" "nixies-us_IN-12"
+		(property "Footprint" "nixies-us:nixies-us-IN-12-DSUB"
 			(at 216.662 364.49 0)
 			(effects
@@
 			)
 		)
-		(property "Footprint" "nixies-us_IN-12"
+		(property "Footprint" "nixies-us:nixies-us-IN-12-DSUB"
 			(at 64.262 364.49 0)
 			(effects
@@
 			)
 		)
-		(property "Footprint" "nixies-us_IN-12"
+		(property "Footprint" "nixies-us:nixies-us-IN-12-DSUB"
 			(at 140.462 364.49 0)
 			(effects
@@
 			)
 		)
-		(property "Footprint" ""
+		(property "Footprint" "NCH8200HV:NCH8200HV"
 			(at 156.21 233.68 0)
 			(effects
@@
 			)
 		)
-		(property "Footprint" ""
+		(property "Footprint" "Resistor_THT:R_Axial_DIN0207_L6.3mm_D2.5mm_P10.16mm_Horizontal"
 			(at 150.622 364.49 90)
 			(effects
@@
 			)
 		)
-		(property "Footprint" ""
+		(property "Footprint" "Resistor_THT:R_Axial_DIN0207_L6.3mm_D2.5mm_P10.16mm_Horizontal"
 			(at 107.442 364.49 90)
 			(effects
@@
 			)
 		)
-		(property "Footprint" "nixies-us_IN-12"
+		(property "Footprint" "nixies-us:nixies-us-IN-12-DSUB"
 			(at 97.282 364.49 0)
 			(effects
@@
 			)
 		)
-		(property "Footprint" "nixies-us_IN-12"
+		(property "Footprint" "nixies-us:nixies-us-IN-12-DSUB"
 			(at 173.482 364.49 0)
 			(effects

Commit message: hardware files update
Parts:
- NX1, NX2, NX3, NX4, NX5, NX6: footprint nixies-us:nixies-us-IN-12-DSUB -> NCH8200HV:IN-12
Connections:
- net A8: now reaches U1.14 (DRAIN4)
- net A8: now also NX1.8
- net A9: now reaches U1.15 (DRAIN5)
- net A9: now also NX1.9
- net A0: now reaches U1.16 (DRAIN6)
- net A0: now also NX1.0
- net A.: now reaches U1.17 (DRAIN7)
- net A.: now also NX1.LHDP
- net A1: now reaches U1.4 (DRAIN0)
- net A1: now also NX1.1
- net A2: now reaches U1.5 (DRAIN1)
- net A2: now also NX1.2
- net A3: now reaches U1.6 (DRAIN2)
- net A3: now also NX1.3
- net A4: now reaches U1.7 (DRAIN3)
- net A4: now also NX1.4
- net A5: now reaches NX1.5
- net A5: now also U2.5 (DRAIN1)
- net A6: now reaches NX1.6
- net A6: now also U2.6 (DRAIN2)
- net A7: now reaches NX1.7
- net A7: now also U2.7 (DRAIN3)
- net B6: now reaches U3.14 (DRAIN4)
- net B6: now also NX2.6
- net B5: now reaches U3.15 (DRAIN5)
- net B5: now also NX2.5
- net B7: now reaches U3.4 (DRAIN0)
- net B7: now also NX2.7
- net B8: now reaches U3.5 (DRAIN1)
- net B8: now also NX2.8
- net B9: now reaches U3.6 (DRAIN2)
- net B9: now also NX2.9
- net B0: now reaches U3.7 (DRAIN3)
- net B0: now also NX2.0
- net B1: now reaches NX2.1
- net B1: now also U2.16 (DRAIN6)
- net B2: now reaches NX2.2
- net B2: now also U2.15 (DRAIN5)
- net B3: now reaches NX2.3
- net B3: now also U2.14 (DRAIN4)
- net B4: now reaches NX2.4
- net B4: now also U2.4 (DRAIN0)
- net B.: now reaches NX2.LHDP
- net B.: now also U2.17 (DRAIN7)

Commit message: hardwareisveryhard
Connections:
- net C7: now reaches U4.14 (DRAIN4)
- net C7: now also NX3.7
- net C8: now reaches U4.15 (DRAIN5)
- net C8: now also NX3.8
- net C9: now reaches U4.16 (DRAIN6)
- net C9: now also NX3.9
- net C0: now reaches U4.17 (DRAIN7)
- net C0: now also NX3.0
- net C.: now reaches U4.4 (DRAIN0)
- net C.: now also NX3.LHDP
- net C1: now reaches U4.5 (DRAIN1)
- net C1: now also NX3.1
- net C2: now reaches U4.6 (DRAIN2)
- net C2: now also NX3.2
- net C3: now reaches U4.7 (DRAIN3)
- net C3: now also NX3.3
- net F0: now reaches NX6.0
- net F0: now also U8.17 (DRAIN7)
- net F1: now reaches NX6.1
- net F1: now also U8.5 (DRAIN1)
- net F2: now reaches NX6.2
- net F2: now also U8.6 (DRAIN2)
- net F3: now reaches NX6.3
- net F3: now also U8.7 (DRAIN3)
- net F4: now reaches NX6.4
- net F4: now also U7.17 (DRAIN7)
- net F5: now reaches NX6.5
- net F5: now also U9.4 (DRAIN0)
- net F6: now reaches NX6.6
- net F6: now also U9.5 (DRAIN1)
- net F7: now reaches NX6.7
- net F7: now also U8.14 (DRAIN4)
- net F8: now reaches NX6.8
- net F8: now also U8.15 (DRAIN5)
- net F9: now reaches NX6.9
- net F9: now also U8.16 (DRAIN6)
- net F.: now reaches NX6.LHDP
- net F.: now also U8.4 (DRAIN0)
- net E0: now reaches NX5.0
- net E0: now also U7.7 (DRAIN3)
- net E1: now reaches NX5.1
- net E1: now also U6.15 (DRAIN5)
- net E2: now reaches NX5.2
- net E2: now also U6.16 (DRAIN6)
- net E3: now reaches NX5.3
- net E3: now also U6.17 (DRAIN7)
- net E4: now reaches NX5.4
- net E4: now also U7.16 (DRAIN6)
- net E5: now reaches NX5.5
- net E5: now also U7.15 (DRAIN5)
- net E6: now reaches NX5.6
- net E6: now also U7.14 (DRAIN4)
- net E7: now reaches NX5.7
- net E7: now also U7.4 (DRAIN0)
- net E8: now reaches NX5.8
- net E8: now also U7.5 (DRAIN1)
- net E9: now reaches NX5.9
- net E9: now also U7.6 (DRAIN2)
- net E.: now reaches NX5.LHDP
- net E.: now also U6.14 (DRAIN4)
- net D7: now reaches U5.14 (DRAIN4)
- net D7: now also NX4.7
- net D8: now reaches U5.15 (DRAIN5)
- net D8: now also NX4.8
- net D9: now reaches U5.16 (DRAIN6)
- net D9: now also NX4.9
- net D0: now reaches U5.17 (DRAIN7)
- net D0: now also NX4.0
- net D1: now reaches U5.4 (DRAIN0)
- net D1: now also NX4.1
- net D2: now reaches U5.5 (DRAIN1)
- net D2: now also NX4.2
- net D.: now reaches U5.6 (DRAIN2)
- net D.: now also NX4.LHDP
- net C6: now reaches U5.7 (DRAIN3)
- net C6: now also NX3.6
- net C4: now reaches NX3.4
- net C4: now also U3.17 (DRAIN7)
- net C5: now reaches NX3.5
- net C5: now also U3.16 (DRAIN6)
- net D3: now reaches U6.4 (DRAIN0)
- net D3: now also NX4.3
- net D4: now reaches U6.5 (DRAIN1)
- net D4: now also NX4.4
- net D5: now reaches U6.6 (DRAIN2)
- net D5: now also NX4.5
- net D6: now reaches U6.7 (DRAIN3)
- net D6: now also NX4.6
